File: sprucep2_left/sprucep2_left.kicad_pcb (KiCad board)
At the start: 2 copper layers, 95.2 x 81 mm, 60 parts, among them J1 USB_C_Receptacle_USB2.0, U1 STM32F072CBT6, U2 PRTR5V0U2X, U3 XC6206PxxxMR-Regulator_Linear, U4 TRRS

Commit message: svgs
Other:
- board text added: "USB"
Changed lines of the file:
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@@
         (effects (font (size 1 1) (thickness 0.15)))
     )
-    (fp_text value "TRRS" (at 0 5.159375 90) (layer "B.Fab")
-        (effects (font (size 1 1) (thickness 0.15)) (justify mirror))
+    (fp_text value "TRRS" (at 0 3.571875 90) (layer "Dwgs.User")
+        (effects (font (size 1 1) (thickness 0.15)))
     )
     (fp_text user "Ring2" (at 0 -3.25 90) (layer "B.Fab")
@@
     (effects (font (size 1 1.5) (thickness 0.25) bold) (justify left bottom mirror))
   )
+  (gr_text "USB" (at 34.76875 10.540625) (layer "Dwgs.User")
+    (effects (font (size 1 1) (thickness 0.15)) (justify left bottom mirror))
+  )
   (segment (start 33.759375 29.978125) (end 33.759375 28.128125) (width 0.4) (layer "B.Cu") (net 1))
