File: sprucep2_right/sprucep2_right.kicad_pcb (KiCad board)
At the start: 2 copper layers, 95.2 x 81 mm, 59 parts, among them J1 USB_C_Receptacle_USB2.0, U1 STM32F072CBT6, U2 PRTR5V0U2X, U3 XC6206PxxxMR-Regulator_Linear, U4 TRRS

Commit message: svgs
Other:
- board text added: "USB"
Changed lines of the file:
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@@
         (effects (font (size 1 1) (thickness 0.15)))
     )
-    (fp_text value "TRRS" (at 0 5.278125 90) (layer "B.Fab")
-        (effects (font (size 1 1) (thickness 0.15)) (justify mirror))
+    (fp_text value "TRRS" (at 0 3.29375 90) (layer "Dwgs.User")
+        (effects (font (size 1 1) (thickness 0.15)))
     )
     (fp_text user "Sleeve" (at 0.25 -11.4 90) (layer "B.Fab")
@@
     (effects (font (size 1 1.5) (thickness 0.25) bold) (justify left bottom mirror))
   )
+  (gr_text "USB" (at 89.934375 11.334375) (layer "Dwgs.User")
+    (effects (font (size 1.5 1.5) (thickness 0.3) bold) (justify left bottom))
+  )
   (segment (start 92.625 30.37375) (end 92.625 28.52375) (width 0.4) (layer "B.Cu") (net 1))
