File: spruce_p3_together/righthalf.kicad_sch (KiCad schematic)
At the start: 22 parts, among them J1 USB_C_Receptacle_USB2.0, U1 STM32F072CBT6, U2 PRTR5V0U2X, U8 TRRS

Commit message: routing for keys
Connections:
- net +3V3 renamed +3.3VA
- net +5V renamed +5VA
- net B1 renamed R_R3
- net B10 renamed R_R1
- net B11 renamed R_R0
- net B2 renamed R_R2
- net B5 renamed R_C0
- net B6 renamed R_C1
- net B7 renamed R_C2
- net B8 renamed R_C3
- net B9 renamed R_C4
