File: spruce_p3_together/spruce_p3_together.kicad_pcb (KiCad board)
At the start: 2 copper layers, 218.5 x 81 mm, 120 parts, among them J1 USB_C_Receptacle_USB2.0, J2 USB_C_Receptacle_USB2.0, U1 STM32F072CBT6, U2 PRTR5V0U2X, U3 XC6206PxxxMR-Regulator_Linear, U4 STM32F072CBT6, U5 PRTR5V0U2X, U6 XC6206PxxxMR-Regulator_Linear, U7 TRRS, U8 TRRS

Commit message: routing for keys
Connections:
- BOOT2 pad 1: +3V3 -> +3.3VA
- C12 pad 1: +3V3 -> +3.3VA
- C13 pad 1: +3V3 -> +3.3VA
- C14 pad 1: +3V3 -> +3.3VA
- C15 pad 1: +3V3 -> +3.3VA
- C16 pad 1: +3V3 -> +3.3VA
- C17 pad 1: +3V3 -> +3.3VA
- C18 pad 1: +5V -> +5VA
- C19 pad 1: +5V -> +5VA
- C20 pad 1: +3V3 -> +3.3VA
- F2 pad 2: +5V -> +5VA
- U1 pad 13: /Left Half/A3 -> L_C0
- U1 pad 14: /Left Half/A4 -> L_C1
- U1 pad 15: /Left Half/A5 -> L_C2
- U1 pad 16: /Left Half/A6 -> L_C3
- U1 pad 17: /Left Half/A7 -> L_C4
- U1 pad 37: /Left Half/A14 -> L_R0
- U1 pad 38: /Left Half/A15 -> L_R1
- U1 pad 39: /Left Half/B3 -> L_R2
- U1 pad 40: /Left Half/B4 -> L_R3
- U4 pad 1: +3V3 -> +3.3VA
- U4 pad 19: /Right Half/B1 -> R_R3
- U4 pad 20: /Right Half/B2 -> R_R2
- U4 pad 21: /Right Half/B10 -> R_R1
- U4 pad 22: /Right Half/B11 -> R_R0
- U4 pad 24: +3V3 -> +3.3VA
- U4 pad 36: +3V3 -> +3.3VA
- U4 pad 41: /Right Half/B5 -> R_C0
- U4 pad 42: /Right Half/B6 -> R_C1
- U4 pad 43: /Right Half/B7 -> R_C2
- U4 pad 45: /Right Half/B8 -> R_C3
- U4 pad 46: /Right Half/B9 -> R_C4
- U4 pad 48: +3V3 -> +3.3VA
- U4 pad 9: +3V3 -> +3.3VA
- U5 pad 4: +5V -> +5VA
- U6 pad 2: +3V3 -> +3.3VA
- U6 pad 3: +5V -> +5VA
- U8 pad 2: +3V3 -> +3.3VA
Routing:
- net L_C4: track 52.7 -> 224.8 mm
- net +3.3VA: track 0.00 -> 137.3 mm, vias 0 -> 7
- net L_RX: track 0.00 -> 126.1 mm, vias 0 -> 2
- net R_C0: track 101.7 -> 224.8 mm, vias 0 -> 1
- net L_C3: track 62.4 -> 177.3 mm, vias 0 -> 1
- net R_C1: track 61.9 -> 176.2 mm
- net L_TX: track 0.00 -> 108.9 mm, vias 0 -> 4
- net R_C2: track 61.9 -> 156.5 mm
- net L_C2: track 61.9 -> 154.5 mm, vias 0 -> 1
- net R_TX: track 0.00 -> 82.5 mm, vias 0 -> 2
- net R_RX: track 0.00 -> 80.0 mm, vias 0 -> 2
- net R_R3: track 4.17 -> 83.6 mm, vias 0 -> 2
- net L_R3: track 4.17 -> 80.8 mm, vias 0 -> 2
- net L_C1: track 52.9 -> 127.0 mm
- net R_R2: track 8.33 -> 63.4 mm, vias 0 -> 2
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